Commit message: update urdf collision

File: humanoid-gym/resources/robots/alexbotmini/urdf/alexbotmini.urdf (robot description, URDF)
Before this commit: robot fftai_grmini, 13 links, 12 joints
Links:
- link base_link: geometry collision box size=0.16 0.2 0.15; visual mesh filename=../meshes/base_link.STL
- link leftlink1: geometry visual mesh filename=../meshes/leftlink1.STL
- link leftlink2: geometry collision box size=0.08 0.15 0.2; visual mesh filename=../meshes/leftlink2.STL
- link leftlink3: geometry collision cylinder length=0.1 radius=0.045; visual mesh filename=../meshes/leftlink3.STL
- link leftlink4: geometry collision box size=0.07 0.1 0.15; visual mesh filename=../meshes/leftlink4.STL
- link leftlink6: geometry collision box size=0.1 0.24 0.01; visual mesh filename=../meshes/leftlink6.STL
- link rightlink1: geometry visual mesh filename=../meshes/rightlink1.STL
- link rightlink2: geometry collision box size=0.08 0.15 0.2; visual mesh filename=../meshes/rightlink2.STL
- link rightlink3: geometry collision cylinder length=0.1 radius=0.045; visual mesh filename=../meshes/rightlink3.STL
- link rightlink4: geometry collision box size=0.07 0.1 0.15; visual mesh filename=../meshes/rightlink4.STL
- link rightlink6: geometry collision box size=0.1 0.24 0.01; visual mesh filename=../meshes/rightlink6.STL
Joints:
- joint leftjoint6: limit lower=-0.3 upper=0.3 effort=30 velocity=130 -> lower=-0.5 upper=0.5 effort=30 velocity=130
- joint rightjoint6: limit lower=-0.3 upper=0.3 effort=30 velocity=130 -> lower=-0.5 upper=0.5 effort=30 velocity=130

Commit message: update urdf

File: humanoid-gym/resources/robots/alexbotmini/urdf/alexbotmini.urdf (robot description, URDF)
Before this commit: robot fftai_grmini, 13 links, 12 joints
Links:
- added link dummy_link
Joints:
- added joint dummy_to_base_link: type fixed, parent dummy_link, child base_link, origin xyz=0 0 0 rpy=0 0 -1.5708

Commit message: 1

File: humanoid-gym/resources/robots/alexbotmini/urdf/alexbotmini.urdf (robot description, URDF)
Before this commit: robot fftai_grmini, 13 links, 12 joints
Links:
- added link dummy_link
- link base_link: geometry collision box size=0.16 0.2 0.15; visual mesh filename=../meshes/base_link.STL
- link leftlink1: geometry visual mesh filename=../meshes/leftlink1.STL
- link leftlink2: geometry collision box size=0.08 0.15 0.2; visual mesh filename=../meshes/leftlink2.STL
- link leftlink3: geometry collision cylinder length=0.1 radius=0.045; visual mesh filename=../meshes/leftlink3.STL
- link leftlink4: geometry collision box size=0.07 0.1 0.15; visual mesh filename=../meshes/leftlink4.STL
- link leftlink6: geometry collision box size=0.1 0.24 0.01; visual mesh filename=../meshes/leftlink6.STL
- link rightlink1: geometry visual mesh filename=../meshes/rightlink1.STL
- link rightlink2: geometry collision box size=0.08 0.15 0.2; visual mesh filename=../meshes/rightlink2.STL
- link rightlink3: geometry collision cylinder length=0.1 radius=0.045; visual mesh filename=../meshes/rightlink3.STL
- link rightlink4: geometry collision box size=0.07 0.1 0.15; visual mesh filename=../meshes/rightlink4.STL
- link rightlink6: geometry collision box size=0.1 0.24 0.01; visual mesh filename=../meshes/rightlink6.STL
Joints:
- added joint dummy_to_base_link: type fixed, parent dummy_link, child base_link, origin xyz=0 0 0 rpy=0 0 -1.5708
- joint leftjoint6: limit lower=-0.3 upper=0.3 effort=30 velocity=130 -> lower=-0.5 upper=0.5 effort=30 velocity=130
- joint rightjoint6: limit lower=-0.3 upper=0.3 effort=30 velocity=130 -> lower=-0.5 upper=0.5 effort=30 velocity=130

Commit message: 1
1

File: humanoid-gym/resources/robots/alexbotmini/urdf/alexbotmini.urdf (robot description, URDF)
Before this commit: robot fftai_grmini, 14 links, 13 joints
Links:
- removed link dummy_link
- link base_link: mass 4 -> 7.35718055319755; geometry collision mesh filename=../meshes/base_link.STL; visual mesh filename=../meshes/base_link.STL
- link leftlink1: mass 0.44393 -> 0.523827453897711; geometry collision mesh filename=../meshes/leftlink1.STL; visual mesh filename=../meshes/leftlink1.STL
- link leftlink2: mass 0.95978 -> 0.959639548121109; geometry collision mesh filename=../meshes/leftlink2.STL; visual mesh filename=../meshes/leftlink2.STL
- link leftlink3: mass 0.81627 -> 0.816268978197084; geometry collision mesh filename=../meshes/leftlink3.STL; visual mesh filename=../meshes/leftlink3.STL
- link leftlink4: mass 1.1424 -> 1.19197432366853; geometry collision mesh filename=../meshes/leftlink4.STL; visual mesh filename=../meshes/leftlink4.STL
- link leftlink5: mass 0.017311 -> 0.0173110583311115; geometry collision mesh filename=../meshes/leftlink5.STL; visual mesh filename=../meshes/leftlink5.STL
- link leftlink6: mass 0.45 -> 0.624059283851391; geometry collision mesh filename=../meshes/leftlink6.STL; visual mesh filename=../meshes/leftlink6.STL
- link rightlink1: mass 0.44393 -> 0.523827457014568; geometry collision mesh filename=../meshes/rightlink1.STL; visual mesh filename=../meshes/rightlink1.STL
- link rightlink2: mass 0.95978 -> 0.95964; geometry collision mesh filename=../meshes/rightlink2.STL; visual mesh filename=../meshes/rightlink2.STL
- link rightlink3: mass 0.81499 -> 0.81499254145314; geometry collision mesh filename=../meshes/rightlink3.STL; visual mesh filename=../meshes/rightlink3.STL
- link rightlink4: mass 1.1424 -> 1.192; geometry collision mesh filename=../meshes/rightlink4.STL; visual mesh filename=../meshes/rightlink4.STL
- link rightlink5: mass 0.017311 -> 0.0173110583311115; geometry collision mesh filename=../meshes/rightlink5.STL; visual mesh filename=../meshes/rightlink5.STL
- link rightlink6: mass 0.45 -> 0.4352; geometry collision mesh filename=../meshes/rightlink6.STL; visual mesh filename=../meshes/rightlink6.STL
Joints:
- removed joint dummy_to_base_link
- joint leftjoint1: origin xyz=-0.10252 0.11412 -0.078592 rpy=0 0 0 -> xyz=-0.091 0.02325 -0.0998 rpy=0 0 0
- joint leftjoint2: axis 0 -1 0 -> 0 1 0; limit lower=-0.3 upper=0.2 effort=51 velocity=59 -> lower=-1 upper=1 effort=51 velocity=59; origin xyz=-0.052 -0.0816 1.2733E-05 rpy=0 0 0 -> xyz=-0.052 -0.081595 0.00093349 rpy=0 0 0
- joint leftjoint3: axis 0. -0. -1 -> 0 0 1; origin xyz=0.0023389 0.077519 -0.15883 rpy=0 0 0 -> xyz=-0.00092023 0.075722 -0.1597 rpy=0 0 0
- joint leftjoint4: axis -1 -0. -0 -> 1 0 0; origin xyz=-0.024903 -0.00058212 -0.14238 rpy=0 0 0 -> xyz=-0.027811 -0.0028522 -0.14181 rpy=0 0 0
- joint leftjoint5: axis -1 -0 -0 -> 0 1 0; origin xyz=0.029296 -0.0057869 -0.28923 rpy=0 0 0 -> xyz=0.021337 -0.0042697 -0.28916 rpy=0 0 0
- joint leftjoint6: axis -0 1 0 -> 1 0 0; limit lower=-0.5 upper=0.5 effort=30 velocity=130 -> lower=-1 upper=1 effort=30 velocity=130
- joint rightjoint1: origin xyz=0.077476 0.11412 -0.078592 rpy=0 0 0 -> xyz=0.091 0.02325 -0.0998 rpy=0 0 0
- joint rightjoint2: axis 0 -1 0 -> 0 1 0; limit lower=-0.2 upper=0.3 effort=51 velocity=59 -> lower=-1 upper=1 effort=51 velocity=59; origin xyz=0.052 -0.081598 0.00059629 rpy=0 0 0 -> xyz=0.052 -0.081599 -0.00047085 rpy=0 0 0
- joint rightjoint3: axis 0 -0 -1 -> 0 0 1; origin xyz=0.0040538 0.077296 -0.1589 rpy=0 0 0 -> xyz=0.001813 0.079368 -0.15792 rpy=0 0 0
- joint rightjoint4: axis 1 -0 0 -> 1 0 0; origin xyz=0.03062 -0.000827 -0.14126 rpy=0 0 0 -> xyz=0.028485 -0.0014832 -0.1417 rpy=0 0 0
- joint rightjoint5: axis 1 -0 0 -> 0 1 0; origin xyz=-0.017523 0.00046354 -0.29026 rpy=0 0 0 -> xyz=-0.02312 -0.010345 -0.28903 rpy=0 0 0
- joint rightjoint6: axis -0 -1 -0 -> -1 0 0; limit lower=-0.5 upper=0.5 effort=30 velocity=130 -> lower=-1 upper=1 effort=30 velocity=130
