Commit message: add some policy
add some policy

File: Alexbotmini_lowerbody/humanoid-gym/resources/robots/alexbotmini/urdf/alexbotmini.urdf (robot description, URDF)
Before this commit: robot fftai_grmini, 14 links, 13 joints
Links:
- link base_link: geometry collision box name=baselink size=0.16 0.2 0.15; visual mesh filename=../meshes/base_link.STL
- link leftlink2: geometry collision box name=left2 size=0.08 0.15 0.2; visual mesh filename=../meshes/leftlink2.STL
- link leftlink3: geometry collision cylinder length=0.1 name=left3 radius=0.045; visual mesh filename=../meshes/leftlink3.STL
- link leftlink4: geometry collision box name=left4 size=0.07 0.1 0.15; visual mesh filename=../meshes/leftlink4.STL
- link leftlink6: geometry collision box name=left6 size=0.1 0.24 0.01; visual mesh filename=../meshes/leftlink6.STL
- link rightlink2: geometry collision box name=right2 size=0.08 0.15 0.2; visual mesh filename=../meshes/rightlink2.STL
- link rightlink3: geometry collision cylinder length=0.1 name=right3 radius=0.045; visual mesh filename=../meshes/rightlink3.STL
- link rightlink4: geometry collision box name=right4 size=0.07 0.1 0.15; visual mesh filename=../meshes/rightlink4.STL
- link rightlink6: geometry collision box name=right6 size=0.1 0.24 0.01; visual mesh filename=../meshes/rightlink6.STL
