Commit message: use new urdf to train
use new urdf to train

File: Lowerbody/humanoid-gym/resources/robots/alexbotmini/urdf/alexbotmini.urdf (robot description, URDF)
Before this commit: robot alexbotmini, 13 links, 12 joints
Links:
- link base_link: mass 4 -> 4.2205; geometry collision box name=baselink size=0.16 0.16 0.12; visual mesh filename=../meshes/base_link.STL
- link leftlink1: mass 0.44393 -> 0.50984
- link leftlink2: mass 0.95978 -> 0.95964; geometry collision box name=leftlink2 size=0.15 0.08 0.20; visual mesh filename=../meshes/leftlink2.STL
- link leftlink3: geometry collision cylinder length=0.1 name=leftlink3 radius=0.045; visual mesh filename=../meshes/leftlink3.STL
- link leftlink4: mass 1.1424 -> 1.192; geometry collision box name=leftlink4 size=0.07 0.08 0.16; visual mesh filename=../meshes/leftlink4.STL
- link leftlink6: mass 0.45 -> 0.62409; geometry collision mesh filename=../meshes/leftlink6.STL; visual mesh filename=../meshes/leftlink6.STL
- link rightlink1: mass 0.44393 -> 0.50984
- link rightlink2: mass 0.95978 -> 0.95964; geometry collision box name=rightlink2 size=0.15 0.08 0.20; visual mesh filename=../meshes/rightlink2.STL
- link rightlink3: geometry collision cylinder length=0.1 name=rightlink3 radius=0.045; visual mesh filename=../meshes/rightlink3.STL
- link rightlink4: mass 1.1424 -> 1.19197938223878; geometry collision box name=rightlink4 size=0.07 0.08 0.16; visual mesh filename=../meshes/rightlink4.STL
- link rightlink5: mass 0.017311 -> 0.019917
- link rightlink6: mass 0.45 -> 0.43259; geometry collision mesh filename=../meshes/rightlink6.STL; visual mesh filename=../meshes/rightlink6.STL
Joints:
- joint leftjoint1: axis -1 0 0 -> 0 1 0; limit lower=-1 upper=1 effort=96 velocity=10.4719755 -> lower=-1 upper=1 effort=96 velocity=12; origin xyz=0 0.095 -0.078592 rpy=0 0 -1.57 -> xyz=0 0.091 -0.08 rpy=0 0 0
- joint leftjoint2: axis 0 -1 0 -> -1 0 0; limit lower=-0.3 upper=0.2 effort=51 velocity=10.4719755 -> lower=-1 upper=1 effort=51 velocity=6.28; origin xyz=-0.052 -0.0816 1.2733E-05 rpy=0 0 0 -> xyz=-0.0816 0.052 -0.0002344 rpy=0 0 0
- joint leftjoint3: axis 0. -0. 1 -> 0 0 -1; limit lower=-1 upper=1 effort=51 velocity=10.4719755 -> lower=-1 upper=1 effort=51 velocity=6.28; origin xyz=0.0023389 0.077519 -0.15883 rpy=0 0 0 -> xyz=0.078 0 -0.15861 rpy=0 0 0
- joint leftjoint4: axis -1 -0. -0 -> 0 1 0; limit lower=-1 upper=1 effort=96 velocity=10.4719755 -> lower=-1 upper=1 effort=96 velocity=12; origin xyz=-0.024903 -0.00058212 -0.14238 rpy=0 0 0 -> xyz=0 0.027 -0.142 rpy=0 0 0
- joint leftjoint5: axis -1 -0 -0 -> 0 -1 0; limit lower=-1 upper=1 effort=30 velocity=13.613568149999999 -> lower=-1 upper=1 effort=30 velocity=14; origin xyz=0.029296 -0.0057869 -0.28923 rpy=0 0 0 -> xyz=-0.0062437 -0.023 -0.289 rpy=0 0 0
- joint leftjoint6: axis -0 1 0 -> 1 0 0; limit lower=-0.5 upper=0.5 effort=30 velocity=13.613568149999999 -> lower=-1 upper=1 effort=30 velocity=14
- joint rightjoint1: axis 1 0 0 -> 0 -1 0; limit lower=-1 upper=1 effort=96 velocity=10.47 -> lower=-1 upper=1 effort=96 velocity=12; origin xyz=0 -0.093 -0.078592 rpy=0 0 -1.57 -> xyz=0 -0.089 -0.08 rpy=0 0 0
- joint rightjoint2: axis 0 -1 0 -> -1 0 0; limit lower=-0.2 upper=0.3 effort=51 velocity=6.178465545 -> lower=-1 upper=1 effort=51 velocity=6.28; origin xyz=0.052 -0.081598 0.00059629 rpy=0 0 0 -> xyz=-0.0816 -0.052 0.0002344 rpy=0 0 0
- joint rightjoint3: axis 0 -0 -1 -> 0 0 -1; limit lower=-1 upper=1 effort=51 velocity=6.178465545 -> lower=-1 upper=1 effort=51 velocity=6.28; origin xyz=0.0040538 0.077296 -0.1589 rpy=0 0 0 -> xyz=0.078 0 -0.15861 rpy=0 0 0
- joint rightjoint4: axis 1 -0 0 -> 0 -1 0; limit lower=-1 upper=1 effort=96 velocity=10.4719755 -> lower=-1 upper=1 effort=96 velocity=12; origin xyz=0.03062 -0.000827 -0.14126 rpy=0 0 0 -> xyz=0 -0.027 -0.142 rpy=0 0 0
- joint rightjoint5: axis 1 -0 0 -> 0 1 0; limit lower=-1 upper=1 effort=30 velocity=13.613568149999999 -> lower=-1 upper=1 effort=30 velocity=14; origin xyz=-0.017523 0.00046354 -0.29026 rpy=0 0 0 -> xyz=-0.0062206 0.025 -0.289 rpy=0 0 0
- joint rightjoint6: axis -0 -1 -0 -> -1 0 0; limit lower=-0.5 upper=0.5 effort=30 velocity=13.613568149999999 -> lower=-1 upper=1 effort=30 velocity=14

Commit message: delete unnecessary package
delete unnecessary package

File: Lowerbody/humanoid-gym/resources/robots/alexbotmini/urdf/alexbotmini.urdf (robot description, URDF)
Before this commit: robot Alexbotmini_lowerbody, 13 links, 12 joints
Links:
- link leftlink6: geometry collision box size=0.1 0.24 0.01; visual mesh filename=../meshes/leftlink6.STL
- link rightlink6: geometry collision box size=0.1 0.24 0.01; visual mesh filename=../meshes/rightlink6.STL
Joints:
- joint leftjoint2: limit lower=-1 upper=1 effort=51 velocity=6.28 -> lower=-1 upper=1 effort=51 velocity=12
- joint leftjoint3: limit lower=-1 upper=1 effort=51 velocity=6.28 -> lower=-1 upper=1 effort=51 velocity=12
- joint leftjoint5: limit lower=-1 upper=1 effort=30 velocity=14 -> lower=-1 upper=1 effort=30 velocity=12
- joint leftjoint6: limit lower=-1 upper=1 effort=30 velocity=14 -> lower=-1 upper=1 effort=30 velocity=12
- joint rightjoint2: limit lower=-1 upper=1 effort=51 velocity=6.28 -> lower=-1 upper=1 effort=51 velocity=12
- joint rightjoint3: limit lower=-1 upper=1 effort=51 velocity=6.28 -> lower=-1 upper=1 effort=51 velocity=12
- joint rightjoint5: limit lower=-1 upper=1 effort=30 velocity=14 -> lower=-1 upper=1 effort=30 velocity=13
- joint rightjoint6: limit lower=-1 upper=1 effort=30 velocity=14 -> lower=-1 upper=1 effort=30 velocity=13

Commit message: add sim2sim
sim2sim done

File: Lowerbody/humanoid-gym/resources/robots/alexbotmini/urdf/alexbotmini.urdf (robot description, URDF)
Before this commit: robot alexbotmini, 13 links, 12 joints
Links:
- link base_link: mass 4.2205 -> 3.703
- link leftlink1: mass 0.50984 -> 1.3062404
- link leftlink2: mass 0.95964 -> 1.7560393
- link leftlink3: mass 0.81627 -> 2.1149564
- link leftlink4: mass 1.192 -> 2.1749387
- link leftlink6: mass 0.62409 -> 0.5
- link rightlink1: mass 0.50984 -> 1.3062404
- link rightlink2: mass 0.95964 -> 1.7560393
- link rightlink3: mass 0.81499 -> 2.115
- link rightlink4: mass 1.19197938223878 -> 2.1749387
- link rightlink5: mass 0.019917 -> 0.017311
- link rightlink6: mass 0.43259 -> 0.5
Joints:
- joint leftjoint1: limit lower=-1 upper=1 effort=96 velocity=12 -> lower=-1 upper=1 effort=96 velocity=20
- joint leftjoint2: limit lower=-1 upper=1 effort=51 velocity=12 -> lower=-1 upper=1 effort=51 velocity=13
- joint leftjoint3: limit lower=-1 upper=1 effort=51 velocity=12 -> lower=-1 upper=1 effort=51 velocity=13
- joint leftjoint4: limit lower=-1 upper=1 effort=96 velocity=12 -> lower=-1 upper=1 effort=96 velocity=20
- joint leftjoint5: limit lower=-1 upper=1 effort=30 velocity=12 -> lower=-1 upper=1 effort=30 velocity=22
- joint leftjoint6: limit lower=-1 upper=1 effort=30 velocity=12 -> lower=-1 upper=1 effort=30 velocity=22
- joint rightjoint1: limit lower=-1 upper=1 effort=96 velocity=12 -> lower=-1 upper=1 effort=96 velocity=20
- joint rightjoint2: limit lower=-1 upper=1 effort=51 velocity=12 -> lower=-1 upper=1 effort=51 velocity=13
- joint rightjoint3: limit lower=-1 upper=1 effort=51 velocity=12 -> lower=-1 upper=1 effort=51 velocity=13
- joint rightjoint4: limit lower=-1 upper=1 effort=96 velocity=12 -> lower=-1 upper=1 effort=96 velocity=20
- joint rightjoint5: limit lower=-1 upper=1 effort=30 velocity=13 -> lower=-1 upper=1 effort=30 velocity=22
- joint rightjoint6: limit lower=-1 upper=1 effort=30 velocity=13 -> lower=-1 upper=1 effort=30 velocity=22

Commit message: add train (after refine)

File: Lowerbody/humanoid-gym/resources/robots/alexbotmini/urdf/alexbotmini.urdf (robot description, URDF)
Before this commit: robot alexbotmini, 13 links, 12 joints
Links:
- link base_link: mass 3.703 -> 5
Joints:
- joint leftjoint1: limit lower=-1 upper=1 effort=96 velocity=20 -> lower=-1 upper=1 effort=96 velocity=10.47
- joint leftjoint2: limit lower=-1 upper=1 effort=51 velocity=13 -> lower=-1 upper=1 effort=51 velocity=6.17
- joint leftjoint3: limit lower=-1 upper=1 effort=51 velocity=13 -> lower=-1 upper=1 effort=51 velocity=6.17
- joint leftjoint4: limit lower=-1 upper=1 effort=96 velocity=20 -> lower=-1 upper=1 effort=96 velocity=10.47
- joint leftjoint5: limit lower=-1 upper=1 effort=30 velocity=22 -> lower=-1 upper=1 effort=30 velocity=13
- joint leftjoint6: limit lower=-1 upper=1 effort=30 velocity=22 -> lower=-0 upper=0 effort=30 velocity=13
- joint rightjoint1: limit lower=-1 upper=1 effort=96 velocity=20 -> lower=-1 upper=1 effort=96 velocity=10.47
- joint rightjoint2: limit lower=-1 upper=1 effort=51 velocity=13 -> lower=-1 upper=1 effort=51 velocity=6.17
- joint rightjoint3: limit lower=-1 upper=1 effort=51 velocity=13 -> lower=-1 upper=1 effort=51 velocity=6.17
- joint rightjoint4: limit lower=-1 upper=1 effort=96 velocity=20 -> lower=-1 upper=1 effort=96 velocity=10.47
- joint rightjoint5: limit lower=-1 upper=1 effort=30 velocity=22 -> lower=-1 upper=1 effort=30 velocity=13.67
- joint rightjoint6: limit lower=-1 upper=1 effort=30 velocity=22 -> lower=-1 upper=1 effort=30 velocity=13.67

Commit message: add train
add train

File: Lowerbody/humanoid-gym/resources/robots/alexbotmini/urdf/alexbotmini.urdf (robot description, URDF)
Before this commit: robot alexbotmini, 13 links, 12 joints
Links:
- link base_link: mass 5 -> 3.703
Joints:
- joint leftjoint6: limit lower=-0 upper=0 effort=30 velocity=13 -> lower=-1 upper=1 effort=30 velocity=13
